File: hw/main_board/kicad_project/_autosave-tDCS_driver.kicad_pcb (KiCad board)
At the start: 2 copper layers, 1 part

Commit message: finalized all footprints for main board, need to pick connectors and finalize stacking desing
Parts:
- removed TQFN_16: VAL**, TQFN-EP_16_5x5mm
Changed lines of the file:
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@@
     (tracks 0)
     (zones 0)
-    (modules 1)
+    (modules 0)
     (nets 1)
   )
@@
     (mod_text_size 1.5 1.5)
     (mod_text_width 0.15)
-    (pad_size 0.35 1)
+    (pad_size 1 0.35)
     (pad_drill 0)
     (pad_to_mask_clearance 0.2)
@@
     (add_net "")
   )
-  (module TQFN-EP_16_5x5mm (layer F.Cu)
-    (at 481.33 90.17)
-    (clearance 0.1)
-    (fp_text reference TQFN_16 (at 7.6 -3.9) (layer F.SilkS)
-      (effects (font (size 1.5 1.5) (thickness 0.15)))
-    )
-    (fp_text value VAL** (at 6.3 4.1) (layer F.SilkS)
-      (effects (font (size 1.5 1.5) (thickness 0.15)))
-    )
-    (fp_line (start -2.5 -2) (end -2 -2.5) (layer F.SilkS) (width 0.15))
-    (fp_line (start -2 -2.5) (end 2.5 -2.5) (layer F.SilkS) (width 0.15))
-    (fp_line (start 2.5 -2.5) (end 2.5 2.5) (layer F.SilkS) (width 0.15))
-    (fp_line (start 2.5 2.5) (end -2.5 2.5) (layer F.SilkS) (width 0.15))
-    (fp_line (start -2.5 2.5) (end -2.5 -2) (layer F.SilkS) (width 0.15))
-    (pad 5 smd rect (at -1.2 2.4 270) (size 0.8 0.25)
-      (layers F.Cu F.Paste F.Mask)
-    )
-    (pad 6 smd rect (at -0.4 2.4 270) (size 0.8 0.25)
-      (layers F.Cu F.Paste F.Mask)
-    )
-    (pad 8 smd rect (at 1.2 2.4 270) (size 0.8 0.25)
-      (layers F.Cu F.Paste F.Mask)
-    )
-    (pad 7 smd rect (at 0.4 2.4 270) (size 0.8 0.25)
-      (layers F.Cu F.Paste F.Mask)
-    )
-    (pad 14 smd rect (at 0.4 -2.4 270) (size 0.8 0.25)
-      (layers F.Cu F.Paste F.Mask)
-    )
-    (pad 13 smd rect (at 1.2 -2.4 270) (size 0.8 0.25)
-      (layers F.Cu F.Paste F.Mask)
-    )
-    (pad 15 smd rect (at -0.4 -2.4 270) (size 0.8 0.25)
-      (layers F.Cu F.Paste F.Mask)
-    )
-    (pad 16 smd rect (at -1.2 -2.4 270) (size 0.8 0.25)
-      (layers F.Cu F.Paste F.Mask)
-    )
-    (pad 12 smd rect (at 2.4 -1.2 180) (size 0.8 0.25)
-      (layers F.Cu F.Paste F.Mask)
-    )
-    (pad 11 smd rect (at 2.4 -0.4 180) (size 0.8 0.25)
-      (layers F.Cu F.Paste F.Mask)
-    )
-    (pad 9 smd rect (at 2.4 1.2 180) (size 0.8 0.25)
-      (layers F.Cu F.Paste F.Mask)
-    )
-    (pad 10 smd rect (at 2.4 0.4 180) (size 0.8 0.25)
-      (layers F.Cu F.Paste F.Mask)
-    )
-    (pad 3 smd rect (at -2.4 0.4 180) (size 0.8 0.25)
-      (layers F.Cu F.Paste F.Mask)
-    )
-    (pad 4 smd rect (at -2.4 1.2 180) (size 0.8 0.25)
-      (layers F.Cu F.Paste F.Mask)
-    )
-    (pad 2 smd rect (at -2.4 -0.4 180) (size 0.8 0.25)
-      (layers F.Cu F.Paste F.Mask)
-    )
-    (pad 1 smd rect (at -2.4 -1.2 180) (size 0.8 0.25)
-      (layers F.Cu F.Paste F.Mask)
-    )
-  )
 )
