File: hw/main_board/kicad_project/_autosave-.kicad_pcb (KiCad board)
At the start: 4 copper layers, 63.5 x 63.5 mm, 77 parts, among them U1 SI5351A, U2 AD5292, U3 AD8221, U4 OP1177, U5 MAX338, U6 MAX338, U7 MAX338, U8 MAX3002, U9 MAX3002, X1 CRYSTAL6-10pf

Commit message: started mainboard pcb layout, fixing small things in schematic, TODO: schematic connector symbols and pads
Parts:
- moved C36 320.0 mm to (352.9, 151.3)
- moved RV6 286.2 mm to (260.1, 265.0)
- moved RV5 285.5 mm to (243.5, 265.6)
- moved RV10 259.0 mm to (260.9, 274.1)
- moved RV3 256.2 mm to (215.6, 266.6)
- moved RV9 255.7 mm to (245.5, 275.8)
- moved RV4 255.0 mm to (228.0, 265.4)
- moved C26 239.4 mm to (201.2, 199.4)
- moved U5 238.7 mm to (222.5, 238.0), turned to 0 degrees
- moved R7 237.5 mm to (195.1, 256.9)
- moved C27 223.3 mm to (203.8, 206.9)
- moved RV8 221.9 mm to (228.3, 274.8)
- moved C25 221.9 mm to (186.1, 201.2)
- moved RV7 221.0 mm to (213.7, 275.2)
- moved R5 216.8 mm to (176.0, 256.9)
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Connections:
- net /CurrentSource/RANGE1 renamed N-0000067
- net /CurrentSource/RANGE2 renamed N-0000060
- net /CurrentSource/RANGE3 renamed N-0000059
- net /CurrentSource/RANGE4 renamed N-0000058
- net /CurrentSource/RANGE5 renamed N-0000071
- net /CurrentSource/RANGE6 renamed N-0000072
- net /CurrentSource/RANGE7 renamed N-0000073
- net /CurrentSource/RANGE8 renamed N-0000074
Other:
- board outline removed
- copper layers 4 -> 2
- net class Inner_signal_8mil removed
- net class Outer_signal_6mil removed
- net class Power removed
- rule trace_min: 0.1524 -> 0.254
