File: hw/main_board/kicad_project/mux.sch (KiCad schematic (older format))
At the start: 12 parts, among them P5 CONN_8, P7 CONN_8, U6 MAX338, U7 MAX338

Commit message: final rework of mux board, finalizing stacking connectors, almost there
Parts:
- removed P5, P7: CONN_8, symbol CONN_8
- added P10, P11, P12, P13, P5, P7, P8, P9: CONN_2, symbol CONN_2
Changed lines of the file:
@@
 EESchema Schematic File Version 2
-LIBS:power
-LIBS:device
-LIBS:transistors
-LIBS:conn
-LIBS:linear
-LIBS:regul
-LIBS:74xx
-LIBS:cmos4000
-LIBS:adc-dac
-LIBS:memory
-LIBS:xilinx
-LIBS:special
-LIBS:microcontrollers
-LIBS:dsp
-LIBS:microchip
-LIBS:analog_switches
-LIBS:motorola
-LIBS:texas
-LIBS:intel
-LIBS:audio
-LIBS:interface
-LIBS:digital-audio
-LIBS:philips
-LIBS:display
-LIBS:cypress
-LIBS:siliconi
-LIBS:opto
-LIBS:atmel
-LIBS:contrib
-LIBS:valves
 LIBS:ddslib
-LIBS:demuxcomplib
-LIBS:tdsc-kicad-convert
 LIBS:tDCS_driver-cache
 EELAYER 24 0
@@
 Comment4 ""
 $EndDescr
-Text Label 8000 5550 0    60   ~ 0
-MUXB7
-Text Label 8000 5150 0    60   ~ 0
-MUXB6
-Text Label 8000 5650 0    60   ~ 0
-MUXB5
-Text Label 8000 5050 0    60   ~ 0
-MUXB4
-Text Label 8000 5750 0    60   ~ 0
-MUXB3
-Text Label 8000 4950 0    60   ~ 0
-MUXB2
-Text Label 8000 5850 0    60   ~ 0
-MUXB1
-Text Label 8000 4850 0    60   ~ 0
-MUXB0
-Text Label 6800 5550 2    60   ~ 0
-MUXA7
-Text Label 6800 5150 2    60   ~ 0
-MUXA6
-Text Label 6800 5650 2    60   ~ 0
-MUXA5
-Text Label 6800 5050 2    60   ~ 0
-MUXA4
-Text Label 6800 5750 2    60   ~ 0
-MUXA3
-Text Label 6800 4950 2    60   ~ 0
-MUXA2
-Text Label 6800 5850 2    60   ~ 0
-MUXA1
-Text Label 6800 4850 2    60   ~ 0
-MUXA0
-$Comp
-L AGND #PWR047
+$Comp
+L AGND #PWR053
 U 1 1 53170BAB
 P 5650 4800
-F 0 "#PWR047" H 5650 4800 40  0001 C CNN
+F 0 "#PWR053" H 5650 4800 40  0001 C CNN
 F 1 "AGND" H 5650 4730 50  0000 C CNN
 F 2 "" H 5650 4800 60  0001 C CNN
@@
 	9600 1750 9700 1850
 $Comp
-L AGND #PWR048
+L AGND #PWR054
 U 1 1 53170CB9
 P 9850 2950
-F 0 "#PWR048" H 9850 2950 40  0001 C CNN
+F 0 "#PWR054" H 9850 2950 40  0001 C CNN
 F 1 "AGND" H 9850 2880 50  0000 C CNN
 F 2 "" H 9850 2950 60  0001 C CNN
@@
 $EndComp
 $Comp
-L AVSS #PWR049
+L AVSS #PWR055
 U 1 1 53170CBF
 P 10950 2050
-F 0 "#PWR049" H 10950 2050 30  0001 C CNN
+F 0 "#PWR055" H 10950 2050 30  0001 C CNN
 F 1 "AVSS" H 10950 1980 30  0000 C CNN
 F 2 "" H 10950 2050 60  0001 C CNN
@@
 $EndComp
 $Comp
-L AVDD #PWR050
+L AVDD #PWR056
 U 1 1 53170CD1
 P 10150 2100
-F 0 "#PWR050" H 10150 2200 30  0001 C CNN
+F 0 "#PWR056" H 10150 2200 30  0001 C CNN
 F 1 "AVDD" H 10150 2210 30  0000 C CNN
 F 2 "" H 10150 2100 60  0001 C CNN
@@
 $EndComp
 $Comp
-L AGND #PWR051
+L AGND #PWR057
 U 1 1 53170CD7
 P 10550 2150
-F 0 "#PWR051" H 10550 2150 40  0001 C CNN
+F 0 "#PWR057" H 10550 2150 40  0001 C CNN
 F 1 "AGND" H 10550 2080 50  0000 C CNN
 F 2 "" H 10550 2150 60  0001 C CNN
@@
 	4500 1450 4600 1550
 $Comp
-L AGND #PWR052
+L AGND #PWR058
 U 1 1 53171190
 P 4750 2650
-F 0 "#PWR052" H 4750 2650 40  0001 C CNN
+F 0 "#PWR058" H 4750 2650 40  0001 C CNN
 F 1 "AGND" H 4750 2580 50  0000 C CNN
 F 2 "" H 4750 2650 60  0001 C CNN
@@
 $EndComp
 $Comp
-L AGND #PWR053
+L AGND #PWR059
 U 1 1 531711A2
 P 5500 1850
-F 0 "#PWR053" H 5500 1850 40  0001 C CNN
+F 0 "#PWR059" H 5500 1850 40  0001 C CNN
 F 1 "AGND" H 5500 1780 50  0000 C CNN
 F 2 "" H 5500 1850 60  0001 C CNN
@@
 $EndComp
 $Comp
-L AVDD #PWR054
+L AVDD #PWR060
 U 1 1 531711A8
 P 5100 1800
-F 0 "#PWR054" H 5100 1900 30  0001 C CNN
+F 0 "#PWR060" H 5100 1900 30  0001 C CNN
 F 1 "AVDD" H 5100 1910 30  0000 C CNN
 F 2 "" H 5100 1800 60  0001 C CNN
@@
 $EndComp
 $Comp
-L AVSS #PWR055
+L AVSS #PWR061
 U 1 1 531711BA
 P 5900 1750
-F 0 "#PWR055" H 5900 1750 30  0001 C CNN
+F 0 "#PWR061" H 5900 1750 30  0001 C CNN
 F 1 "AVSS" H 5900 1680 30  0000 C CNN
 F 2 "" H 5900 1750 60  0001 C CNN
@@
 Text Label 9500 1500 2    60   ~ 0
 OUT_MUX[0...3]
-Text Label 9650 5200 0    60   ~ 0
+Text Label 10400 4650 2    60   ~ 0
 MUXB7
-Text Label 9650 5100 0    60   ~ 0
+Text Label 8650 4650 2    60   ~ 0
 MUXB6
-Text Label 9650 5000 0    60   ~ 0
+Text Label 10400 4250 2    60   ~ 0
 MUXB5
-Text Label 9650 4900 0    60   ~ 0
+Text Label 10400 3800 2    60   ~ 0
 MUXB4
-Text Label 9650 4800 0    60   ~ 0
+Text Label 9550 4250 2    60   ~ 0
 MUXB3
-Text Label 9650 4700 0    60   ~ 0
+Text Label 9550 3800 2    60   ~ 0
 MUXB2
-Text Label 9650 4600 0    60   ~ 0
+Text Label 8650 4250 2    60   ~ 0
 MUXB1
-Text Label 9650 4500 0    60   ~ 0
+Text Label 8650 3800 2    60   ~ 0
 MUXB0
-Text Label 9650 6100 0    60   ~ 0
+Text Label 10400 4450 2    60   ~ 0
 MUXA7
-Text Label 9650 6000 0    60   ~ 0
+Text Label 8650 4450 2    60   ~ 0
 MUXA6
-Text Label 9650 5900 0    60   ~ 0
+Text Label 10400 4050 2    60   ~ 0
 MUXA5
-Text Label 9650 5800 0    60   ~ 0
+Text Label 10400 3600 2    60   ~ 0
 MUXA4
-Text Label 9650 5700 0    60   ~ 0
+Text Label 9550 4050 2    60   ~ 0
 MUXA3
-Text Label 9650 5600 0    60   ~ 0
+Text Label 9550 3600 2    60   ~ 0
 MUXA2
-Text Label 9650 5500 0    60   ~ 0
+Text Label 8650 4050 2    60   ~ 0
 MUXA1
-Text Label 9650 5400 0    60   ~ 0
+Text Label 8650 3600 2    60   ~ 0
 MUXA0
-$Comp
-L CONN_8 P7
-U 1 1 53171513
-P 10000 5750
-F 0 "P7" V 9950 5750 60  0000 C CNN
-F 1 "CONN_8" V 10050 5750 60  0000 C CNN
-F 2 "" H 10000 5750 60  0001 C CNN
-F 3 "" H 10000 5750 60  0001 C CNN
-	1    10000 5750
-	1    0    0    -1
-$EndComp
-$Comp
-L CONN_8 P5
-U 1 1 53171519
-P 10000 4850
-F 0 "P5" V 9950 4850 60  0000 C CNN
-F 1 "CONN_8" V 10050 4850 60  0000 C CNN
-F 2 "" H 10000 4850 60  0001 C CNN
-F 3 "" H 10000 4850 60  0001 C CNN
-	1    10000 4850
-	1    0    0    -1
-$EndComp
 Text HLabel 7400 2750 1    60   Input ~ 0
 I_IN
@@
 Connection ~ 5100 1800
 Connection ~ 4900 1550
+$Comp
+L CONN_2 P5
+U 1 1 531FA735
+P 9000 3700
+F 0 "P5" V 8950 3700 40  0000 C CNN
+F 1 "CONN_2" V 9050 3700 40  0000 C CNN
+F 2 "" H 9000 3700 60  0000 C CNN
+F 3 "" H 9000 3700 60  0000 C CNN
+	1    9000 3700
+	1    0    0    -1
+$EndComp
+$Comp
+L CONN_2 P7
+U 1 1 531FA746
+P 9000 4150
+F 0 "P7" V 8950 4150 40  0000 C CNN
+F 1 "CONN_2" V 9050 4150 40  0000 C CNN
+F 2 "" H 9000 4150 60  0000 C CNN
+F 3 "" H 9000 4150 60  0000 C CNN
+	1    9000 4150
+	1    0    0    -1
+$EndComp
+$Comp
+L CONN_2 P9
+U 1 1 531FA74C
+P 9900 3700
+F 0 "P9" V 9850 3700 40  0000 C CNN
+F 1 "CONN_2" V 9950 3700 40  0000 C CNN
+F 2 "" H 9900 3700 60  0000 C CNN
+F 3 "" H 9900 3700 60  0000 C CNN
+	1    9900 3700
+	1    0    0    -1
+$EndComp
+$Comp
+L CONN_2 P10
+U 1 1 531FA752
+P 9900 4150
+F 0 "P10" V 9850 4150 40  0000 C CNN
+F 1 "CONN_2" V 9950 4150 40  0000 C CNN
+F 2 "" H 9900 4150 60  0000 C CNN
+F 3 "" H 9900 4150 60  0000 C CNN
+	1    9900 4150
+	1    0    0    -1
+$EndComp
+$Comp
+L CONN_2 P11
+U 1 1 531FA758
+P 10750 3700
+F 0 "P11" V 10700 3700 40  0000 C CNN
+F 1 "CONN_2" V 10800 3700 40  0000 C CNN
+F 2 "" H 10750 3700 60  0000 C CNN
+F 3 "" H 10750 3700 60  0000 C CNN
+	1    10750 3700
+	1    0    0    -1
+$EndComp
+$Comp
+L CONN_2 P12
+U 1 1 531FA75E
+P 10750 4150
+F 0 "P12" V 10700 4150 40  0000 C CNN
+F 1 "CONN_2" V 10800 4150 40  0000 C CNN
+F 2 "" H 10750 4150 60  0000 C CNN
+F 3 "" H 10750 4150 60  0000 C CNN
+	1    10750 4150
+	1    0    0    -1
+$EndComp
+$Comp
+L CONN_2 P13
+U 1 1 531FA764
+P 10750 4550
+F 0 "P13" V 10700 4550 40  0000 C CNN
+F 1 "CONN_2" V 10800 4550 40  0000 C CNN
+F 2 "" H 10750 4550 60  0000 C CNN
+F 3 "" H 10750 4550 60  0000 C CNN
+	1    10750 4550
+	1    0    0    -1
+$EndComp
+$Comp
+L CONN_2 P8
+U 1 1 531FA76A
+P 9000 4550
+F 0 "P8" V 8950 4550 40  0000 C CNN
+F 1 "CONN_2" V 9050 4550 40  0000 C CNN
+F 2 "" H 9000 4550 60  0000 C CNN
+F 3 "" H 9000 4550 60  0000 C CNN
+	1    9000 4550
+	1    0    0    -1
+$EndComp
+Text Label 8000 4850 0    60   ~ 0
+MUXA0
+Text Label 8000 4950 0    60   ~ 0
+MUXA1
+Text Label 8000 5050 0    60   ~ 0
+MUXA2
+Text Label 8000 5150 0    60   ~ 0
+MUXA3
+Text Label 6800 4850 2    60   ~ 0
+MUXA4
+Text Label 6800 4950 2    60   ~ 0
+MUXA5
+Text Label 6800 5050 2    60   ~ 0
+MUXA6
+Text Label 6800 5150 2    60   ~ 0
+MUXA7
+Text Label 8000 5850 0    60   ~ 0
+MUXB0
+Text Label 8000 5750 0    60   ~ 0
+MUXB1
+Text Label 8000 5650 0    60   ~ 0
+MUXB2
+Text Label 8000 5550 0    60   ~ 0
+MUXB3
+Text Label 6800 5850 2    60   ~ 0
+MUXB4
+Text Label 6800 5750 2    60   ~ 0
+MUXB5
+Text Label 6800 5650 2    60   ~ 0
+MUXB6
+Text Label 6800 5550 2    60   ~ 0
+MUXB7
 $EndSCHEMATC

Commit message: finished component layout on mainboard, need to route power planes and the digital control signal lines
Changed lines of the file:
@@
 EESchema Schematic File Version 2
 LIBS:ddslib
+LIBS:demuxcomplib
 LIBS:tDCS_driver-cache
 EELAYER 24 0
@@
 $EndDescr
 $Comp
-L AGND #PWR053
+L AGND #PWR052
 U 1 1 53170BAB
 P 5650 4800
-F 0 "#PWR053" H 5650 4800 40  0001 C CNN
+F 0 "#PWR052" H 5650 4800 40  0001 C CNN
 F 1 "AGND" H 5650 4730 50  0000 C CNN
 F 2 "" H 5650 4800 60  0001 C CNN
@@
 	9600 1750 9700 1850
 $Comp
-L AGND #PWR054
+L AGND #PWR053
 U 1 1 53170CB9
 P 9850 2950
-F 0 "#PWR054" H 9850 2950 40  0001 C CNN
+F 0 "#PWR053" H 9850 2950 40  0001 C CNN
 F 1 "AGND" H 9850 2880 50  0000 C CNN
 F 2 "" H 9850 2950 60  0001 C CNN
@@
 $EndComp
 $Comp
-L AVSS #PWR055
+L AVSS #PWR054
 U 1 1 53170CBF
 P 10950 2050
-F 0 "#PWR055" H 10950 2050 30  0001 C CNN
+F 0 "#PWR054" H 10950 2050 30  0001 C CNN
 F 1 "AVSS" H 10950 1980 30  0000 C CNN
 F 2 "" H 10950 2050 60  0001 C CNN
@@
 $EndComp
 $Comp
-L AVDD #PWR056
+L AVDD #PWR055
 U 1 1 53170CD1
 P 10150 2100
-F 0 "#PWR056" H 10150 2200 30  0001 C CNN
+F 0 "#PWR055" H 10150 2200 30  0001 C CNN
 F 1 "AVDD" H 10150 2210 30  0000 C CNN
 F 2 "" H 10150 2100 60  0001 C CNN
@@
 $EndComp
 $Comp
-L AGND #PWR057
+L AGND #PWR056
 U 1 1 53170CD7
 P 10550 2150
-F 0 "#PWR057" H 10550 2150 40  0001 C CNN
+F 0 "#PWR056" H 10550 2150 40  0001 C CNN
 F 1 "AGND" H 10550 2080 50  0000 C CNN
 F 2 "" H 10550 2150 60  0001 C CNN
@@
 	4500 1450 4600 1550
 $Comp
-L AGND #PWR058
+L AGND #PWR057
 U 1 1 53171190
 P 4750 2650
-F 0 "#PWR058" H 4750 2650 40  0001 C CNN
+F 0 "#PWR057" H 4750 2650 40  0001 C CNN
 F 1 "AGND" H 4750 2580 50  0000 C CNN
 F 2 "" H 4750 2650 60  0001 C CNN
@@
 $EndComp
 $Comp
-L AGND #PWR059
+L AGND #PWR058
 U 1 1 531711A2
 P 5500 1850
-F 0 "#PWR059" H 5500 1850 40  0001 C CNN
+F 0 "#PWR058" H 5500 1850 40  0001 C CNN
 F 1 "AGND" H 5500 1780 50  0000 C CNN
 F 2 "" H 5500 1850 60  0001 C CNN
@@
 $EndComp
 $Comp
-L AVDD #PWR060
+L AVDD #PWR059
 U 1 1 531711A8
 P 5100 1800
-F 0 "#PWR060" H 5100 1900 30  0001 C CNN
+F 0 "#PWR059" H 5100 1900 30  0001 C CNN
 F 1 "AVDD" H 5100 1910 30  0000 C CNN
 F 2 "" H 5100 1800 60  0001 C CNN
@@
 $EndComp
 $Comp
-L AVSS #PWR061
+L AVSS #PWR060
 U 1 1 531711BA
 P 5900 1750
-F 0 "#PWR061" H 5900 1750 30  0001 C CNN
+F 0 "#PWR060" H 5900 1750 30  0001 C CNN
 F 1 "AVSS" H 5900 1680 30  0000 C CNN
 F 2 "" H 5900 1750 60  0001 C CNN
@@
 F 3 "" H 10750 3700 60  0000 C CNN
 	1    10750 3700
-	1    0    0    -1
+	1    0    0    1
 $EndComp
 $Comp
@@
 F 3 "" H 10750 4150 60  0000 C CNN
 	1    10750 4150
-	1    0    0    -1
+	1    0    0    1
 $EndComp
 $Comp
@@
 F 3 "" H 10750 4550 60  0000 C CNN
 	1    10750 4550
-	1    0    0    -1
+	1    0    0    1
 $EndComp
 $Comp
@@
 F 3 "" H 9000 4550 60  0000 C CNN
 	1    9000 4550
-	1    0    0    -1
+	1    0    0    1
 $EndComp
 Text Label 8000 4850 0    60   ~ 0
@@
 Text Label 6800 5150 2    60   ~ 0
 MUXA7
+Text Label 8000 5550 0    60   ~ 0
+MUXB0
+Text Label 8000 5650 0    60   ~ 0
+MUXB1
+Text Label 8000 5750 0    60   ~ 0
+MUXB2
 Text Label 8000 5850 0    60   ~ 0
-MUXB0
-Text Label 8000 5750 0    60   ~ 0
-MUXB1
-Text Label 8000 5650 0    60   ~ 0
-MUXB2
-Text Label 8000 5550 0    60   ~ 0
 MUXB3
+Text Label 6800 5550 2    60   ~ 0
+MUXB4
+Text Label 6800 5650 2    60   ~ 0
+MUXB5
+Text Label 6800 5750 2    60   ~ 0
+MUXB6
 Text Label 6800 5850 2    60   ~ 0
-MUXB4
-Text Label 6800 5750 2    60   ~ 0
-MUXB5
-Text Label 6800 5650 2    60   ~ 0
-MUXB6
-Text Label 6800 5550 2    60   ~ 0
 MUXB7
 $EndSCHEMATC
