File: hw/main_board/kicad_project/tDCS_driver.kicad_pcb (KiCad board)
At the start: 4 copper layers, 63.5 x 63.5 mm, 77 parts, among them U1 SI5351A, U2 AD5292, U3 AD8221, U4 OP1177, U5 MAX338, U6 MAX338, U7 MAX338, U8 MAX3002, U9 MAX3002, X1 CRYSTAL6-10pf

Commit message: final rework of mux board, finalizing stacking connectors, almost there
Parts:
- added P1: CONN_5, SIL-5, F.Cu at (134.6, -36.8)
- added P10: CONN_2, MOLEX_SL_2_PCB, F.Cu at (439.2, 67.2)
- added P11: CONN_2, MOLEX_SL_2_PCB, F.Cu at (494.4, 43.4)
- added P12: CONN_2, MOLEX_SL_2_PCB, F.Cu at (457.3, 67.2)
- added P13: CONN_2, MOLEX_SL_2_PCB, F.Cu at (489.3, 66.3)
- added P2: CONN_5, SIL-5, F.Cu at (149.9, -36.8)
- added P3: CONN_6, SIL-6, F.Cu at (196.8, -45.7)
- added P4: CONN_3X2, MOLEX_MEGAFIT_6, F.Cu at (-36.6, 26.4)
- added P5: CONN_2, MOLEX_SL_2_PCB, F.Cu at (513.7, 64.3)
- added P6: CONN_20X2, HEAD_50P_Vert_0.1, F.Cu at (-96.9, 14.4)
- added P7: CONN_2, MOLEX_SL_2_PCB, F.Cu at (424.6, 40.5)
- added P8: CONN_2, MOLEX_SL_2_PCB, F.Cu at (437.0, 40.8)
- added P9: CONN_2, MOLEX_SL_2_PCB, F.Cu at (471.8, 41.1)
- U1: footprint QSOP_16 -> MSOP-10
- U2: footprint MSOP-10 -> TSSOP_14
- U3: footprint TSSOP_14 -> MSOP_8
- moved RV3 379.3 mm to (301.0, 94.0), turned to 90 degrees
- moved R5 378.1 mm to (299.7, 87.6)
- moved RV5 367.9 mm to (275.6, 94.0), turned to 90 degrees
- moved R7 366.9 mm to (274.3, 87.6)
- moved RV4 356.3 mm to (288.3, 94.0), turned to 90 degrees
- moved R6 354.2 mm to (287.0, 87.6)
- moved RV6 343.9 mm to (262.9, 94.0), turned to 90 degrees
- moved R8 342.0 mm to (261.6, 87.6)
- moved RV10 340.0 mm to (294.6, 106.7), turned to 270 degrees
- moved RV9 339.2 mm to (281.9, 106.7), turned to 270 degrees
- moved R12 333.9 mm to (293.4, 113.0)
- moved R11 333.0 mm to (280.7, 113.0)
- moved C26 307.1 mm to (242.6, 106.7), turned to 180 degrees
- moved C25 302.8 mm to (242.6, 109.2), turned to 180 degrees
- moved RV7 302.5 mm to (256.5, 106.7), turned to 270 degrees
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Connections:
- net N-0000047 renamed /DDS/DDS_REFOUT
- net N-0000072 renamed /CurrentSource/DPOT_A
- net N-0000073 renamed /CurrentSource/instr_ref
- C4 pad 2: N-0000048 -> /DDS/DDS_DCAP
- C5 pad 1: N-0000049 -> /DDS/DDS_COMP
- C8 pad 2: N-0000050 -> /DDS/DDS_FSADJ
- DDS1 pad 18: N-0000050 -> /DDS/DDS_FSADJ
- DDS1 pad 20: N-0000049 -> /DDS/DDS_COMP
- DDS1 pad 3: N-0000048 -> /DDS/DDS_DCAP
- DDS1 pad EP: (no net) -> AGND
- R1 pad 1: N-0000050 -> /DDS/DDS_FSADJ
- R1 pad 2: N-0000051 -> N-0000043
- R10 pad 2: N-0000053 -> N-0000050
- R11 pad 2: N-0000056 -> N-0000051
- R12 pad 2: N-0000057 -> N-0000052
- R4 pad 1: N-0000058 -> /CurrentSource/Rg1
- R5 pad 2: N-0000054 -> N-0000044
- R6 pad 2: N-0000055 -> N-0000045
- R7 pad 2: N-0000066 -> N-0000046
- R8 pad 2: N-0000065 -> N-0000048
- R9 pad 2: N-0000052 -> N-0000049
- U2 pad 4: N-0000071 (its old number) -> /CurrentSource/DPOT_W
- U2 pad 5: N-0000071 (its old number) -> /CurrentSource/DPOT_W
- U3 pad 2: N-0000070 (its old number) -> /CurrentSource/Rg1
- U3 pad 3: N-0000058 -> /CurrentSource/RG2
- U3 pad 7: N-0000069 (its old number) -> /CurrentSource/AD8211_IOUT
- U5 pad 8: N-0000069 (its old number) -> /CurrentSource/AD8211_IOUT
- U6 pad 10: /OutputMultiplexer/MUXA4 -> /OutputMultiplexer/MUXA6
- U6 pad 11: /OutputMultiplexer/MUXA2 -> /OutputMultiplexer/MUXA5
- U6 pad 12: /OutputMultiplexer/MUXA0 -> /OutputMultiplexer/MUXA4
- U6 pad 4: /OutputMultiplexer/MUXB0 -> /OutputMultiplexer/MUXA0
- U6 pad 5: /OutputMultiplexer/MUXB2 -> /OutputMultiplexer/MUXA1
- U6 pad 6: /OutputMultiplexer/MUXB4 -> /OutputMultiplexer/MUXA2
- U6 pad 7: /OutputMultiplexer/MUXB6 -> /OutputMultiplexer/MUXA3
- U6 pad 9: /OutputMultiplexer/MUXA6 -> /OutputMultiplexer/MUXA7
- U7 pad 10: /OutputMultiplexer/MUXA5 -> /OutputMultiplexer/MUXB6
- U7 pad 11: /OutputMultiplexer/MUXA3 -> /OutputMultiplexer/MUXB5
- U7 pad 12: /OutputMultiplexer/MUXA1 -> /OutputMultiplexer/MUXB4
- U7 pad 4: /OutputMultiplexer/MUXB1 -> /OutputMultiplexer/MUXB0
- U7 pad 5: /OutputMultiplexer/MUXB3 -> /OutputMultiplexer/MUXB1
- U7 pad 6: /OutputMultiplexer/MUXB5 -> /OutputMultiplexer/MUXB2
- U7 pad 7: /OutputMultiplexer/MUXB7 -> /OutputMultiplexer/MUXB3
- U7 pad 9: /OutputMultiplexer/MUXA7 -> /OutputMultiplexer/MUXB7
Routing:
- net /CurrentSource/IOUT: track 0.00 -> 111.5 mm
- net AGND: track 0.00 -> 93.8 mm, vias 0 -> 6
- net /CurrentSource/RANGE8: track 0.00 -> 64.3 mm
- net /CurrentSource/RANGE1: track 0.00 -> 58.3 mm
- net /CurrentSource/RANGE7: track 0.00 -> 50.3 mm
- net /CurrentSource/RANGE2: track 0.00 -> 44.3 mm
- net /CurrentSource/RANGE6: track 0.00 -> 36.3 mm
- net /CurrentSource/RANGE3: track 0.00 -> 30.3 mm
- net /CurrentSource/RANGE5: track 0.00 -> 22.4 mm
- net AVDD: track 0.00 -> 20.3 mm
- net AVSS: track 0.00 -> 20.3 mm
- net /CurrentSource/DPOT_W: track 0.00 -> 17.8 mm
- net /CurrentSource/RANGE4: track 0.00 -> 16.3 mm
- net N-0000043: track 0.00 -> 15.1 mm
- net /DDS/VOut-: track 0.00 -> 11.4 mm
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- added copper zone on GND, net AGND
Other:
- board outline removed
- net class Power: via_dia 0.889 -> 1.27
- net class Primary_Signal added: clearance 0.381, trace_width 0.254, via_dia 0.889, via_drill 0.635
- rule via_min_drill: 0.508 -> 0.2921
- rule via_min_size: 0.889 -> 0.8001

Commit message: finished component layout on mainboard, need to route power planes and the digital control signal lines
Parts:
- removed P1, P2: CONN_5, SIL-5
- removed P3: CONN_6, SIL-6
- added P14: CONN_5X2, HEADER-2x5-SAMTEC, F.Cu at (261.6, 109.2)
- added P15: CONN_5X2, HEADER-2x5-SAMTEC, F.Cu at (292.1, 109.2)
- added P16: CONN_3X2, HEADER-2x3-SAMTEC, F.Cu at (276.9, 109.2)
- added P17: CONN_2X2, HEADER-2x2-SAMTEC, F.Cu at (302.3, 99.7)
- added P18: CONN_2X2, HEADER-2x2-SAMTEC, F.Cu at (302.3, 118.7)
- added SCREW1: CONN_1, SCREW_3mm, F.Cu at (245.1, 90.2)
- added SCREW2: CONN_1, SCREW_3mm, F.Cu at (308.6, 128.3)
- added SCREW3: CONN_1, SCREW_3mm, F.Cu at (308.6, 90.2)
- added SCREW4: CONN_1, SCREW_3mm, F.Cu at (245.1, 128.3)
- C1, C11, C12, C13, C14, C15, C16, C17, C18, C19, C2, C20, C21, C22, C23, C24, C25, C26, C27, C28, C29, C3, C30, C31, C32, C33, C34, C4, C43, C44, C5, C6, C7, U8, U9: moved to B.Cu
- moved P6 325.1 mm to (202.6, 141.0)
- moved P5 250.5 mm to (264.2, 86.4)
- moved P11 246.7 mm to (264.2, 132.1), turned to 180 degrees
- moved U8 229.6 mm to (259.1, 121.9), turned to 90 degrees
- moved P4 220.7 mm to (181.0, 63.5), turned to 270 degrees
- moved U9 219.3 mm to (259.1, 96.5), turned to 270 degrees
- moved P13 198.3 mm to (302.3, 132.1), turned to 180 degrees
- moved P12 191.8 mm to (276.9, 132.1), turned to 180 degrees
- moved P9 187.8 mm to (289.6, 86.4)
- moved P8 173.4 mm to (289.6, 132.1), turned to 180 degrees
- moved P7 154.7 mm to (276.9, 86.4)
- moved P10 138.2 mm to (302.3, 86.4)
- moved C39 132.1 mm to (67.6, -101.3)
- moved C41 132.1 mm to (68.0, -97.2)
- moved C42 132.1 mm to (59.7, -83.4)
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Connections:
- P11 pad 1: /OutputMultiplexer/MUXA4 -> /OutputMultiplexer/MUXB4
- P11 pad 2: /OutputMultiplexer/MUXB4 -> /OutputMultiplexer/MUXA4
- P12 pad 1: /OutputMultiplexer/MUXA5 -> /OutputMultiplexer/MUXB5
- P12 pad 2: /OutputMultiplexer/MUXB5 -> /OutputMultiplexer/MUXA5
- P13 pad 1: /OutputMultiplexer/MUXA7 -> /OutputMultiplexer/MUXB7
- P13 pad 2: /OutputMultiplexer/MUXB7 -> /OutputMultiplexer/MUXA7
- P8 pad 1: /OutputMultiplexer/MUXA6 -> /OutputMultiplexer/MUXB6
- P8 pad 2: /OutputMultiplexer/MUXB6 -> /OutputMultiplexer/MUXA6
- R10 pad 1: /CurrentSource/RANGE3 -> N-0000071
- R10 pad 2: N-0000050 (its old number) -> /CurrentSource/IOUT
- R11 pad 1: /CurrentSource/RANGE2 -> N-0000069
- R11 pad 2: N-0000051 (its old number) -> /CurrentSource/IOUT
- R12 pad 1: /CurrentSource/RANGE1 -> N-0000070
- R12 pad 2: N-0000052 (its old number) -> /CurrentSource/IOUT
- R5 pad 1: /CurrentSource/RANGE8 -> N-0000082
- R5 pad 2: N-0000044 -> /CurrentSource/IOUT
- R6 pad 1: /CurrentSource/RANGE7 -> N-0000063
- R6 pad 2: N-0000045 -> /CurrentSource/IOUT
- R7 pad 1: /CurrentSource/RANGE6 -> N-0000062
- R7 pad 2: N-0000046 -> /CurrentSource/IOUT
- R8 pad 1: /CurrentSource/RANGE5 -> N-0000061
- R8 pad 2: N-0000048 (its old number) -> /CurrentSource/IOUT
- R9 pad 1: /CurrentSource/RANGE4 -> N-0000060
- R9 pad 2: N-0000049 (its old number) -> /CurrentSource/IOUT
- RV10 pad 1: N-0000052 (its old number) -> /CurrentSource/RANGE1
- RV10 pad 2: N-0000052 (its old number) -> /CurrentSource/RANGE1
- RV10 pad 3: /CurrentSource/IOUT -> N-0000070
- RV3 pad 1: N-0000044 -> N-0000082
- RV3 pad 2: N-0000044 -> /CurrentSource/RANGE8
- RV3 pad 3: /CurrentSource/IOUT -> /CurrentSource/RANGE8
- RV4 pad 1: N-0000045 -> N-0000063
- RV4 pad 2: N-0000045 -> /CurrentSource/RANGE7
- RV4 pad 3: /CurrentSource/IOUT -> /CurrentSource/RANGE7
- RV5 pad 1: N-0000046 -> N-0000062
- RV5 pad 2: N-0000046 -> /CurrentSource/RANGE6
- RV5 pad 3: /CurrentSource/IOUT -> /CurrentSource/RANGE6
- RV6 pad 1: N-0000048 (its old number) -> N-0000061
- RV6 pad 2: N-0000048 (its old number) -> /CurrentSource/RANGE5
- RV6 pad 3: /CurrentSource/IOUT -> /CurrentSource/RANGE5
- RV7 pad 1: N-0000049 (its old number) -> /CurrentSource/RANGE4
- RV7 pad 2: N-0000049 (its old number) -> /CurrentSource/RANGE4
- RV7 pad 3: /CurrentSource/IOUT -> N-0000060
- RV8 pad 1: N-0000050 (its old number) -> /CurrentSource/RANGE3
- RV8 pad 2: N-0000050 (its old number) -> /CurrentSource/RANGE3
- RV8 pad 3: /CurrentSource/IOUT -> N-0000071
- RV9 pad 1: N-0000051 (its old number) -> /CurrentSource/RANGE2
- RV9 pad 2: N-0000051 (its old number) -> /CurrentSource/RANGE2
- RV9 pad 3: /CurrentSource/IOUT -> N-0000069
- U1 pad 2: N-0000071 -> N-0000084
- U1 pad 3: N-0000070 -> N-0000087
- U1 pad 8: (no net) -> AGND
- U5 pad 1: /CurrentSource/RNG_2 -> /CurrentSource/RNG_1
- U5 pad 13: AVSS -> AVDD
- U5 pad 15: /CurrentSource/RNG_0 -> /CurrentSource/RNG_3
- U5 pad 16: /CurrentSource/RNG_1 -> /CurrentSource/RNG_2
- U5 pad 2: /CurrentSource/RNG_3 -> /CurrentSource/RNG_0
- U5 pad 3: AVDD -> AVSS
- U7 pad 10: /OutputMultiplexer/MUXB6 -> /OutputMultiplexer/MUXB5
- U7 pad 11: /OutputMultiplexer/MUXB5 -> /OutputMultiplexer/MUXB6
- U7 pad 12: /OutputMultiplexer/MUXB4 -> /OutputMultiplexer/MUXB7
- U7 pad 4: /OutputMultiplexer/MUXB0 -> /OutputMultiplexer/MUXB3
- U7 pad 5: /OutputMultiplexer/MUXB1 -> /OutputMultiplexer/MUXB2
- U7 pad 6: /OutputMultiplexer/MUXB2 -> /OutputMultiplexer/MUXB1
- U7 pad 7: /OutputMultiplexer/MUXB3 -> /OutputMultiplexer/MUXB0
- U7 pad 9: /OutputMultiplexer/MUXB7 -> /OutputMultiplexer/MUXB4
- U8 pad 12: /MUXCOM0 -> /MUXC4
- U8 pad 13: /MUXCOM1 -> /MUXC3
- U8 pad 14: /MUXCOM2 -> /MUXC2
- U8 pad 15: /MUXC4 -> /MUXC1
- U8 pad 16: /MUXC3 -> /MUXC0
- U8 pad 17: /MUXC2 -> /MUXCOM0
- U8 pad 18: /MUXC1 -> /MUXCOM2
- U8 pad 20: /MUXC0 -> /MUXCOM1
- X1 pad 1: N-0000071 -> N-0000087
- X1 pad 2: N-0000070 -> N-0000084
Routing:
- net AVSS: track 20.3 -> 224.9 mm, vias 0 -> 6
- net AVDD: track 20.3 -> 216.7 mm, vias 0 -> 6
- net /DDS/DDS_BUS1: track 0.00 -> 114.3 mm, vias 0 -> 1
- net /LogicTranslators/UCOUT7: track 0.00 -> 104.9 mm
- net AVDD_3V3: track 0.00 -> 103.2 mm, vias 0 -> 5
- net /DDS/DDS_BUS2: track 0.00 -> 100.0 mm, vias 0 -> 1
- net /LogicTranslators/UCOUT8: track 0.00 -> 98.0 mm
- net /LogicTranslators/UCOUT0: track 0.00 -> 84.3 mm
- net /LogicTranslators/OUT_MUX1: track 0.00 -> 83.0 mm, vias 0 -> 1
- net /OutputMultiplexer/MUXA7: track 0.00 -> 82.7 mm
- net /OutputMultiplexer/MUXA3: track 0.00 -> 79.8 mm
- net /DDS/DDS_BUS5: track 0.00 -> 70.6 mm, vias 0 -> 1
- net /OutputMultiplexer/MUXA6: track 0.00 -> 68.6 mm
- net /OutputMultiplexer/MUXA2: track 0.00 -> 65.6 mm
- net /MUXD4: track 0.00 -> 64.1 mm
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- added copper zone on B.Cu, net AGND
- added copper zone on F.Cu, net AGND
Other:
- board outline added: 149.9 x 99.1 mm
- net class Inner_signal_8mil removed
- net class Logic added: clearance 0.1524, trace_width 2.032, via_dia 0.889, via_drill 0.381
- net class Outer_signal_6mil removed
- net class Power: via_dia 1.27 -> 1.016; via_drill 0.635 -> 0.508
- net class Primary_Signal removed
- net class Signal added: clearance 0.1524, trace_width 0.254, via_dia 1.016, via_drill 0.508
- rule via_min_drill: 0.2921 -> 0.3048
- rule via_min_size: 0.8001 -> 0.4064

Commit message: Converting keepnote notes to thorough design documentation, starting with BRD1
Parts:
- removed C35, C36, C39, C40: 1uF, 0603
- P6: value CONN_20X2 -> CONN_25X2
- moved C42 288.1 mm to (257.8, 125.7), turned to 90 degrees
- moved C38 284.7 mm to (257.8, 118.1), turned to 270 degrees
- moved C37 284.1 mm to (261.7, 98.6), turned to 90 degrees
- moved C41 270.3 mm to (260.4, 92.7), turned to 270 degrees
- moved U8 25.4 mm to (259.1, 96.5)
- moved U9 25.4 mm to (259.1, 121.9)
- moved C11 5.99 mm to (203.2, 80.0), turned to 270 degrees
- moved C12 5.99 mm to (200.7, 80.0), turned to 270 degrees
- moved P6 4.84 mm to (207.0, 139.1)
- moved C33 2.11 mm to (280.7, 100.3)
- moved C34 2.05 mm to (283.2, 100.3)
- moved C16 1.42 mm to (189.2, 123.2)
- moved C23 1.27 mm to (204.5, 116.8)
Connections:
- P18 pad 1: /MUXVSS -> /powergen/MUXVSS
- P18 pad 2: /MUXVSS -> /powergen/MUXVSS
- P18 pad 3: /MUXVDD -> DVDD_2V5
- P18 pad 4: /MUXVDD -> DVDD_2V5
- P6 pad 1: /LogicTranslators/UCOUT0 -> /Clock/CLK_TWI0
- P6 pad 10: /Clock/CLK_TWI1 -> /CurrentSource/GAIN_BUS1
- P6 pad 11: /LogicTranslators/UCOUT5 -> /CurrentSource/GAIN_BUS2
- P6 pad 12: /DDS/DDS_BUS0 -> /CurrentSource/GAIN_BUS3
- P6 pad 13: /LogicTranslators/UCOUT6 -> /CurrentSource/GAIN_BUS4
- P6 pad 14: /DDS/DDS_BUS1 -> /CurrentSource/GAIN_BUS0
- P6 pad 15: /LogicTranslators/UCOUT7 -> /LogicTranslators/UCOUT14
- P6 pad 16: /DDS/DDS_BUS2 -> /LogicTranslators/UCOUT15
- P6 pad 17: /LogicTranslators/UCOUT8 -> /LogicTranslators/UCOUT16
- P6 pad 18: /DDS/DDS_BUS3 -> /LogicTranslators/UCOUT17
- P6 pad 19: /LogicTranslators/UCOUT9 -> /LogicTranslators/UCOUT18
- P6 pad 2: /LogicTranslators/OUT_MUX1 -> /Clock/CLK_TWI1
- P6 pad 20: /DDS/DDS_BUS4 -> /CurrentSource/RNG_3
- P6 pad 21: /LogicTranslators/UCOUT10 -> /CurrentSource/RNG_2
- P6 pad 22: /DDS/DDS_BUS5 -> /CurrentSource/RNG_1
- P6 pad 23: /LogicTranslators/UCOUT11 -> /CurrentSource/RNG_0
- P6 pad 24: /DDS/DDS_BUS6 -> /LogicTranslators/IN_MUX2
- P6 pad 25: /LogicTranslators/UCOUT12 -> /LogicTranslators/IN_MUX3
- P6 pad 26: /CurrentSource/RNG_0 -> /LogicTranslators/IN_MUX0
- P6 pad 27: /LogicTranslators/UCOUT13 -> /LogicTranslators/IN_MUX1
- P6 pad 28: /CurrentSource/RNG_1 -> /LogicTranslators/UCOUT27
- P6 pad 29: /LogicTranslators/UCOUT14 -> /LogicTranslators/UCOUT28
- P6 pad 3: /LogicTranslators/UCOUT1 -> /DDS/DDS_BUS3
- P6 pad 30: /CurrentSource/RNG_2 -> /LogicTranslators/UCOUT29
- P6 pad 31: /LogicTranslators/IN_MUX0 -> /LogicTranslators/UCOUT30
- P6 pad 32: /CurrentSource/RNG_3 -> /LogicTranslators/UCOUT31
- P6 pad 33: /LogicTranslators/IN_MUX1 -> /LogicTranslators/UCOUT32
- P6 pad 34: /CurrentSource/GAIN_BUS0 -> /LogicTranslators/UCOUT33
- P6 pad 35: /LogicTranslators/IN_MUX2 -> /LogicTranslators/UCOUT34
- P6 pad 36: /CurrentSource/GAIN_BUS1 -> /LogicTranslators/OUT_MUX0
- P6 pad 37: /LogicTranslators/IN_MUX3 -> /LogicTranslators/OUT_MUX1
- P6 pad 38: /CurrentSource/GAIN_BUS2 -> /LogicTranslators/OUT_MUX2
- P6 pad 39: /LogicTranslators/OUT_MUX0 -> /LogicTranslators/OUT_MUX3
- P6 pad 4: /LogicTranslators/OUT_MUX2 -> /DDS/DDS_BUS4
- P6 pad 40: /CurrentSource/GAIN_BUS3 -> /LogicTranslators/UCOUT39
- P6 pad 41: (no net) -> /LogicTranslators/UCOUT40
- P6 pad 42: (no net) -> /LogicTranslators/UCOUT41
- P6 pad 43: (no net) -> /LogicTranslators/UCOUT42
- P6 pad 44: (no net) -> /LogicTranslators/UCOUT43
- P6 pad 45: (no net) -> /LogicTranslators/UCOUT44
- P6 pad 46: (no net) -> /LogicTranslators/UCOUT45
- P6 pad 47: (no net) -> /LogicTranslators/UCOUT46
- P6 pad 48: (no net) -> /LogicTranslators/UCOUT47
- P6 pad 49: (no net) -> /LogicTranslators/UCOUT48
- P6 pad 5: /LogicTranslators/UCOUT2 -> /DDS/DDS_BUS5
- P6 pad 50: (no net) -> /LogicTranslators/UCOUT49
- P6 pad 6: /LogicTranslators/OUT_MUX3 -> /DDS/DDS_BUS6
- P6 pad 7: /LogicTranslators/UCOUT3 -> /DDS/DDS_BUS0
- P6 pad 8: /Clock/CLK_TWI0 -> /DDS/DDS_BUS1
- P6 pad 9: /LogicTranslators/UCOUT4 -> /DDS/DDS_BUS2
- U2 pad 14: /CurrentSource/GAIN_BUS3 -> /CurrentSource/GAIN_BUS4
- U8 pad 1: /LogicTranslators/UCOUT0 -> /MUXD0
- U8 pad 10: /LogicTranslators/UCOUT8 -> N-0000052
- U8 pad 11: AGND -> N-0000061
- U8 pad 12: /MUXC4 -> N-0000050
- U8 pad 13: /MUXC3 -> N-0000049
- U8 pad 14: /MUXC2 -> N-0000048
- U8 pad 15: /MUXC1 -> /LogicTranslators/UCOUT18
- U8 pad 16: /MUXC0 -> /LogicTranslators/UCOUT17
- U8 pad 17: /MUXCOM0 -> /LogicTranslators/UCOUT16
- U8 pad 18: /MUXCOM2 -> /LogicTranslators/UCOUT15
- U8 pad 19: DVDD_2V5 -> AVDD_3V3
- U8 pad 2: AVDD_3V3 -> DVDD_2V5
- U8 pad 20: /MUXCOM1 -> /LogicTranslators/UCOUT14
- U8 pad 3: /LogicTranslators/UCOUT1 -> /MUXD1
- U8 pad 4: /LogicTranslators/UCOUT2 -> /MUXD2
- U8 pad 5: /LogicTranslators/UCOUT3 -> /MUXD3
- U8 pad 6: /LogicTranslators/UCOUT4 -> /MUXD4
- U8 pad 7: /LogicTranslators/UCOUT5 -> N-0000047
- U8 pad 8: /LogicTranslators/UCOUT6 -> N-0000053
- U8 pad 9: /LogicTranslators/UCOUT7 -> N-0000051
- U9 pad 1: N-0000050 -> /MUXC4
- U9 pad 10: /LogicTranslators/UCOUT9 -> N-0000046
- U9 pad 12: /MUXD0 -> /LogicTranslators/UCOUT34
- U9 pad 13: /MUXD1 -> /LogicTranslators/UCOUT33
- U9 pad 14: /MUXD2 -> /LogicTranslators/UCOUT32
- U9 pad 15: /MUXD3 -> /LogicTranslators/UCOUT31
- U9 pad 16: /MUXD4 -> /LogicTranslators/UCOUT30
- U9 pad 17: N-0000048 -> /LogicTranslators/UCOUT29
- U9 pad 18: N-0000047 -> /LogicTranslators/UCOUT28
- U9 pad 19: DVDD_2V5 -> AVDD_3V3
- U9 pad 2: AVDD_3V3 -> DVDD_2V5
- U9 pad 20: N-0000049 -> /LogicTranslators/UCOUT27
- U9 pad 3: N-0000051 -> /MUXC3
- U9 pad 4: N-0000052 -> /MUXC2
- U9 pad 5: /LogicTranslators/UCOUT14 -> /MUXC1
- U9 pad 6: /LogicTranslators/UCOUT13 -> /MUXC0
- U9 pad 7: /LogicTranslators/UCOUT12 -> /MUXCOM0
- U9 pad 8: /LogicTranslators/UCOUT11 -> /MUXCOM2
- U9 pad 9: /LogicTranslators/UCOUT10 -> /MUXCOM1
Routing:
- net AGND: track 55.7 -> 1018.8 mm, vias 16 -> 83
- net AVDD_3V3: track 103.2 -> 520.5 mm, vias 5 -> 10
- net /LogicTranslators/OUT_MUX0: track 4.63 -> 185.8 mm
- net DVDD_2V5: track 0.00 -> 166.0 mm, vias 0 -> 7
- net /LogicTranslators/UCOUT14: track 0.00 -> 114.2 mm
- net /LogicTranslators/OUT_MUX2: track 52.6 -> 165.8 mm
- net /LogicTranslators/UCOUT16: track 0.00 -> 107.4 mm
- net /LogicTranslators/UCOUT15: track 0.00 -> 107.1 mm
- net /LogicTranslators/UCOUT7: track 104.9 -> 0.00 mm
- net /LogicTranslators/OUT_MUX3: track 50.4 -> 155.2 mm
- net /LogicTranslators/UCOUT18: track 0.00 -> 101.8 mm
- net /LogicTranslators/UCOUT17: track 0.00 -> 101.5 mm
- net /LogicTranslators/UCOUT8: track 98.0 -> 0.00 mm
- net /LogicTranslators/OUT_MUX1: track 83.0 -> 176.0 mm
- net /LogicTranslators/UCOUT0: track 84.3 -> 0.00 mm
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- added copper zone on B.Cu, net /powergen/MUXVSS
- added copper zone on F.Cu, net /powergen/MUXVSS
- added copper zone on PWR, net /powergen/MUXVSS
- added copper zone on PWR, net AGND
- added copper zone on B.Cu, net AVDD
- added copper zone on F.Cu, net AVDD
- added copper zone on PWR, net AVDD
- added copper zone on B.Cu, net AVDD_3V3
- added copper zone on F.Cu, net AVDD_3V3
- added copper zone on PWR, net AVDD_3V3
- added copper zone on B.Cu, net AVSS
- added copper zone on F.Cu, net AVSS
- added copper zone on PWR, net AVSS
- added copper zone on B.Cu, net DVDD_2V5
- added copper zone on F.Cu, net DVDD_2V5
- added copper zone on PWR, net DVDD_2V5
Other:
- outline, holes or cut-outs redrawn
- board text added: "(C) 2014 ANDREY SHMAKOV"
- board text added: "TDCS BRD1 1.0 REVA"
