File: hw/main_board/kicad_project/$noname.sch (KiCad schematic (older format))
At the start: 18 parts

Commit message: forgot to add files in last commit
Parts:
- removed C1 (x2), C2 (x2), C3 (x2), C6 (x2), C7 (x2), C8 (x2), C9 (x2): 6u, symbol C
- removed C4 (x2), C5 (x2): 4u, symbol C
- added P? (x8): CONN_2, symbol CONN_2
- added U? (x2): MAX338, QSOP_16, symbol MAX338
Connections:
- net labels added: AGND, I_IN, MUXA0, MUXA1, MUXA2, MUXA3, MUXA4, MUXA5, MUXA6, MUXA7, MUXB0, MUXB1, MUXB2, MUXB3, MUXB4, MUXB5, MUXB6, MUXB7
- net labels removed: A, B
- wire segments 24 -> 2
