File: hw/main_board/kicad_project/figuresch/currentstage.sch (KiCad schematic (older format))
At the start: 32 parts

Commit message: forgot to add files in last commit
Parts:
- removed R?: 2K, symbol R
- removed R?: 5K, symbol R
- removed R?: 10K, symbol R
- removed R?: 22K, symbol R
- removed R?: 45K, symbol R
- removed R?: 91K, symbol R
- removed R?: 182K, symbol R
- removed R?: 374K, symbol R
- removed RV? (x2): 2K, symbol POT
- removed RV? (x3): 5K, symbol POT
- removed RV?: 10K, symbol POT
- removed RV? (x2): 20K, symbol POT
- removed U?: MAX338, symbol MAX338
- added R3: RSET, symbol R
- gave numbers to parts that had none: 14
Connections:
- wire segments 90 -> 43
Other:
- note removed: "0.5uA-1uA"
- note removed: "16uA-32uA"
- note removed: "1uA-2uA"
- note removed: "2uA-4uA"
- note removed: "32uA-64uA"
- note removed: "4uA-8uA"
- note removed: "64uA-100uA"
- note removed: "8uA-16uA"
- note removed: "Output Range Selector"
- moved on the sheet: C7, C8, U3
